File: EBike CAD/Electrical/Control Board/ESP32.sch (KiCad schematic (older format))
At the start: 14 parts, among them J2 Conn_01x05_Female, J3 Conn_01x04_Female, J4 Conn_01x02_Female, J5 Conn_01x03_Female, J6 Conn_01x04_Female, J7 0022232041, SW1 SW_Push

Commit message: fix
Parts:
- gave numbers to parts that had none: 1
Changed lines of the file:
@@
 SCL
 $Comp
-L Connector:Conn_01x04_Female J?
+L Connector:Conn_01x04_Female J12
 U 1 1 5F0A362F
 P 1700 1400
-F 0 "J?" V 1638 1112 50  0000 R CNN
+F 0 "J12" V 1638 1112 50  0000 R CNN
 F 1 "Conn_01x04_Female" V 1547 1112 50  0000 R CNN
 F 2 "Connector_JST:JST_XH_B4B-XH-AM_1x04_P2.50mm_Vertical" H 1700 1400 50  0001 C CNN
@@
 3v3
 $Comp
-L power:GND #PWR?
+L power:GND #PWR0104
 U 1 1 5F0A4397
 P 1900 1600
-F 0 "#PWR?" H 1900 1350 50  0001 C CNN
+F 0 "#PWR0104" H 1900 1350 50  0001 C CNN
 F 1 "GND" H 1905 1427 50  0000 C CNN
 F 2 "" H 1900 1600 50  0001 C CNN
