File: EBike CAD/Electrical/Control Board/Power.sch (KiCad schematic (older format))
At the start: 6 parts, among them J1 Conn_01x02_Female, U1 TL2575HV-33IKTTR

Commit message: fix
Parts:
- U1: footprint Package_TO_SOT_SMD:TO-263-6 -> Package_TO_SOT_SMD:TO-263-5_TabPin6
Changed lines of the file:
@@
 F 0 "U1" H 4650 2187 60  0000 C CNN
 F 1 "TL2575HV-33IKTTR" H 4650 2081 60  0000 C CNN
-F 2 "Package_TO_SOT_SMD:TO-263-6" H 4650 2040 60  0001 C CNN
+F 2 "Package_TO_SOT_SMD:TO-263-5_TabPin6" H 4650 2040 60  0001 C CNN
 F 3 "" H 3250 1800 60  0000 C CNN
 	1    3250 1800
